File: esp32-4-channel-relays.kicad_sch (KiCad schematic)
At the start: 63 parts, among them J1 Relay-1, J2 Relay-2, J3 Relay-3, J4 Relay-4, K1 SRD-05VDC-SL-C, K2 SRD-05VDC-SL-C, K3 SRD-05VDC-SL-C, K4 SRD-05VDC-SL-C, Q1 MBT3904DW1, Q2 BC547A, Q3 BC547A, Q4 BC547A, Q5 BC547A, SW1 SW_SKQG, SW2 SW_SKQG, U1 AMS1117-3.3, U2 CH340C, U3 PRTR5V0U2X, U4 ESP32-WROOM-32, U5 PC817, U6 PC817, U7 PC817, U8 PC817

Commit message: Reconnect relays to esp32 considering footprint placement
Connections:
- net IO_19: now also D4.1 (K); no longer D6.1 (K)
- net IO_21: now also D2.1 (K); no longer D8.1 (K)
- net IO_5: now reaches U4.29 (IO5)
- net IO_5: now also D8.1 (K)
- net IO_18: now reaches U4.30 (IO18)
- net IO_18: now also D6.1 (K)
- net IO_22: no longer names the net of U4.36 (IO22)
- net IO_22: no longer D4.1 (K)
- net IO_23: no longer names the net of U4.37 (IO23)
- net IO_23: no longer D2.1 (K)
Changed lines of the file:
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@@
   (no_connect (at 93.98 166.37))
   (no_connect (at 179.07 43.18))
-  (no_connect (at 93.98 140.97))
   (no_connect (at 93.98 130.81))
   (no_connect (at 63.5 118.11))
@@
   (no_connect (at 93.98 156.21))
   (no_connect (at 63.5 143.51))
-  (no_connect (at 93.98 123.19))
   (no_connect (at 93.98 125.73))
   (no_connect (at 63.5 146.05))
   (no_connect (at 93.98 158.75))
+  (no_connect (at 93.98 148.59))
   (no_connect (at 39.37 161.29))
+  (no_connect (at 93.98 151.13))
   (wire (pts (xy 229.87 163.83) (xy 229.87 167.64))
     (stroke (width 0) (type default))
@@
     (stroke (width 0) (type default))
   )
-  (wire (pts (xy 93.98 151.13) (xy 100.33 151.13))
-    (stroke (width 0) (type default))
-  )
   (wire (pts (xy 24.13 35.56) (xy 24.13 39.37))
     (stroke (width 0) (type default))
@@
     (stroke (width 0) (type default))
   )
+  (wire (pts (xy 93.98 140.97) (xy 100.33 140.97))
+    (stroke (width 0) (type default))
+  )
   (wire (pts (xy 279.4 120.65) (xy 279.4 119.38))
     (stroke (width 0) (type default))
@@
     (stroke (width 0) (type default))
   )
+  (wire (pts (xy 93.98 123.19) (xy 100.33 123.19))
+    (stroke (width 0) (type default))
+  )
   (wire (pts (xy 234.95 158.75) (xy 226.06 158.75))
     (stroke (width 0) (type default))
@@
   )
   (wire (pts (xy 250.19 161.29) (xy 250.19 167.64))
-    (stroke (width 0) (type default))
-  )
-  (wire (pts (xy 93.98 148.59) (xy 100.33 148.59))
     (stroke (width 0) (type default))
   )
@@
     (effects (font (size 1.27 1.27) bold) (justify right bottom))
   )
-  (label "IO_22" (at 116.84 153.67 180) (fields_autoplaced)
+  (label "IO_19" (at 116.84 153.67 180) (fields_autoplaced)
     (effects (font (size 1.27 1.27)) (justify right bottom))
   )
@@
     (effects (font (size 1.27 1.27)) (justify left bottom))
   )
-  (label "IO_23" (at 116.84 107.95 180) (fields_autoplaced)
+  (label "IO_21" (at 116.84 107.95 180) (fields_autoplaced)
     (effects (font (size 1.27 1.27)) (justify right bottom))
   )
@@
     (effects (font (size 1.27 1.27)) (justify left bottom))
   )
-  (label "IO_22" (at 100.33 148.59 0) (fields_autoplaced)
-    (effects (font (size 1.27 1.27)) (justify left bottom))
-  )
   (label "NO-4" (at 298.45 120.65 0) (fields_autoplaced)
     (effects (font (size 1.27 1.27)) (justify left bottom))
   )
-  (label "IO_21" (at 219.71 135.89 180) (fields_autoplaced)
+  (label "IO_5" (at 219.71 135.89 180) (fields_autoplaced)
     (effects (font (size 1.27 1.27)) (justify right bottom))
   )
-  (label "IO_23" (at 100.33 151.13 0) (fields_autoplaced)
+  (label "IO_18" (at 100.33 140.97 0) (fields_autoplaced)
     (effects (font (size 1.27 1.27)) (justify left bottom))
   )
@@
     (effects (font (size 1.27 1.27) bold) (justify right bottom))
   )
-  (label "IO_19" (at 116.84 199.39 180) (fields_autoplaced)
+  (label "IO_18" (at 116.84 199.39 180) (fields_autoplaced)
     (effects (font (size 1.27 1.27)) (justify right bottom))
   )
@@
     (effects (font (size 1.27 1.27)) (justify left bottom))
   )
+  (label "IO_5" (at 100.33 123.19 0) (fields_autoplaced)
+    (effects (font (size 1.27 1.27)) (justify left bottom))
+  )
