File: esp32-4-channel-relays.kicad_sch (KiCad schematic)
At the start: 63 parts, among them J1 Relay-1, J2 Relay-2, J3 Relay-3, J4 Relay-4, K1 SRD-05VDC-SL-C, K2 SRD-05VDC-SL-C, K3 SRD-05VDC-SL-C, K4 SRD-05VDC-SL-C, Q1 MBT3904DW1, Q2 BC547A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

Commit message: Update page setting
Other:
- company: (none) -> Self-Employed
Changed lines of the file:
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@@
     (title "ESP32 4 Channel Relays")
     (date "2023-03-19")
+    (company "Self-Employed")
   )
   (junction (at 45.72 48.26) (diameter 0) (color 0 0 0 0)
